File: interface_temperature/electronique/kicad/LightKitV2/LightKitV2.sch (KiCad schematic (older format))
At the start: 20 parts, among them J1 Conn_01x02, J2 Conn_01x03, J3 Conn_01x02, J4 Conn_01x02, Q1 S8050, Q2 S8050, SW1 SW_SPDT, SW2 SW_Push_Dual, U1 AMS1117-3.3, U2 ESP-01v090

Commit message: Passage en Rev. B du schéma de LightKitV2
Parts:
- added U3: NodeMCU_1.0_(ESP-12E), symbol kicad-ESP8266-master:NodeMCU_1.0_(ESP-12E)
Connections:
- net +5V: now also U3.15 (VIN)
- net GND: now also U3.14 (GND)
- net LED_CMD: now also U3.29 (D1(GPIO5))
- net LED_CMD_DIRECT: now reaches J4.2 (Pin_2), R7.1
- net LED_CMD_DIRECT: now also U3.28 (D2(GPIO4))
- no-connect marks 0 -> 26
Other:
- note added: "*Warning: connect only one microcontroller !"
- note added: "Cut in Rev. B"
- note added: "Microcontroler*"
- note added: "Microcontroller*"
- note added: "Prog is done by\nusing USB"
- note removed: "Microcontroler"
- moved on the sheet: C1, C2, C3, J1, J2, J3, J4, Q1, Q2, R1, R2, R3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
